Commit message: update bunker URDF and bunker

File: bunker_explorer_bot/bunker_explorer_description/urdf/.ipynb_checkpoints/bunker_camera_base-footprint-checkpoint.xacro (robot description, xacro)
@@ -3,7 +3,76 @@
      Commit Version: 1.6.0-1-g15f4949  Build Version: 1.6.7594.29634
      For more information, please see http://wiki.ros.org/sw_urdf_exporter -->
-<robot  name="bunker_description" xmlns:xacro="http://www.ros.org/wiki/xacro">
-  <link
-    name="base_link">
+<robot  name="bunker_realsense_description" xmlns:xacro="http://www.ros.org/wiki/xacro">
+  <xacro:property name="r200_cam_rgb_px" value="0.005"/>
+  <xacro:property name="r200_cam_rgb_py" value="0.018"/>
+  <xacro:property name="r200_cam_rgb_pz" value="0.013"/>
+  <xacro:property name="r200_cam_depth_offset" value="0.01"/>
+  <xacro:arg name="camera_visual" default="false"/>
+  <link name="base_footprint"/>
+  <joint name="base_joint" type="fixed">
+    <parent link="robot_base"/>
+    <child link="base_footprint" /> <!--original: base_link -->
+    <origin xyz="0 0 0.355" rpy="0 0 0"/>
+  </joint>
+<!-- add frame stand joint 13Nov23 -->
+  <joint name="baseto_framestand" type="fixed">
+    <origin rpy="0 0 0" xyz="0.3 0 0"/>
+    <parent link="robot_base"/>
+    <child link="rbot_base2"/>
+  </joint>
+<!-- add maeterial colour for frame stand -->
+  <material name="blue">
+    <color rgba="0 0 0.8 1"/>
+  </material>
+  <material name="red">
+    <color rgba="1 0 0 1"/>
+  </material>
+  <material name="white">
+    <color rgba="1 1 1 1"/>
+  </material>
+  <link name="rbot_base2">
+    <visual>
+      <geometry>
+        <box size="0.045 0.09 0.03"/>
+      </geometry>
+      <origin rpy="0 0 0" xyz="0 0 0"/>
+      <material name="red"/>
+    </visual>
+  </link>
+  <link name="servo_bottom2">
+    <visual>
+      <geometry>
+        <cylinder length="0.25" radius="0.015"/>
+      </geometry>
+      <origin rpy="0 0 0" xyz="0 0 0"/>
+      <material name="green"/>
+    </visual>
+  </link>
+  <link name="up_mount2">
+    <visual>
+      <geometry>
+        <box size="0.05 0.148 0.05"/>
+      </geometry>
+      <origin rpy="0 0. 0" xyz="0 0 0"/>
+      <material name="blue"/>
+    </visual>
+  </link>
+ <joint name="base_to_Servo_B2" type="fixed">
+    <parent link="rbot_base2"/>
+    <child link="servo_bottom2"/>
+    <origin xyz="0 0 0.14"/>
+  </joint>
+ <joint name="servo_bottom_to_up_mount2" type="fixed">
+    <parent link="servo_bottom2"/>
+    <child link="up_mount2"/>
+    <origin xyz="0 0 0.15"/>
+  </joint>
+  <joint name="mount_to_camera2" type="fixed">
+    <parent link="up_mount2"/>
+    <child link="camera_link"/> <!-- original: base_link -->
+    <origin rpy="0 0 0" xyz="0.03 -0.065 0.00"/>
+  </joint>
+  <link
+    name="robot_base"> <!--original : base_link -->
      <inertial>
       <origin
@@ -11,5 +80,5 @@
         rpy="0 0 0" />
       <mass
-        value="22" />
+        value="0.0001" />
       <inertia
         ixx="0.607716166684979"
@@ -29,7 +98,7 @@
       </geometry>
       <material
-        name="Gray">
-        <color
-          rgba="0.5 0.5 0.5 1" />
+        name="">
+        <color
+          rgba="0.5 0.5 0.5  1" />
       </material>
     </visual>
@@ -51,5 +120,5 @@
         rpy="0 0 0" />
       <mass
-        value="0.392034219968119" />
+        value="0.0001" />
       <inertia
         ixx="0.000378440530116381"
@@ -91,5 +160,5 @@
       rpy="1.5708 0 -3.1416" />
     <parent
-      link="base_link" />
+      link="robot_base" /> <!--original base_link -->
     <child
       link="wheel1_Link" />
@@ -109,5 +178,5 @@
         rpy="0 0 0" />
       <mass
-        value="0.190328287901002" />
+        value="0.0001" />
       <inertia
         ixx="6.58750963981394E-05"
@@ -149,5 +218,5 @@
       rpy="1.5708 0 -3.1416" />
     <parent
-      link="base_link" />
+      link="robot_base" /> <!-- original : base_link -->
     <child
       link="wheel1.1_Link" />
@@ -167,5 +236,5 @@
         rpy="0 0 0" />
       <mass
-        value="0.271192811687251" />
+        value="0.0001" />
       <inertia
         ixx="0.000179574259018481"
@@ -207,5 +276,5 @@
       rpy="1.5708 0 -3.1416" />
     <parent
-      link="base_link" />
+      link="robot_base" /> <!-- original : base_link -->
     <child
       link="wheel1.2_Link" />
@@ -225,5 +294,5 @@
         rpy="0 0 0" />
       <mass
-        value="0.245835028330933" />
+        value="0.0001" />
       <inertia
         ixx="0.000105254202004996"
@@ -265,5 +334,5 @@
       rpy="1.5708 0 -3.1416" />
     <parent
-      link="base_link" />
+      link="robot_base" /> <!-- original : base_link -->
     <child
       link="wheel1.3_Link" />
@@ -283,5 +352,5 @@
         rpy="0 0 0" />
       <mass
-        value="0.392034219968119" />
+        value="0.0001" />
       <inertia
         ixx="0.000378440530116381"
@@ -323,5 +392,5 @@
       rpy="1.5708 0 -3.1416" />
     <parent
-      link="base_link" />
+      link="robot_base" /> <!-- original : base_link -->
     <child
       link="wheel2_Link" />
@@ -341,5 +410,5 @@
         rpy="0 0 0" />
       <mass
-        value="0.190328287901002" />
+        value="0.0001" />
       <inertia
         ixx="6.58750963981394E-05"
@@ -381,5 +450,5 @@
       rpy="1.5708 0 -3.1416" />
     <parent
-      link="base_link" />
+      link="robot_base" /> <!-- original : base_link -->
     <child
       link="wheel2.1_Link" />
@@ -399,5 +468,5 @@
         rpy="0 0 0" />
       <mass
-        value="0.27119281168725" />
+        value="0.0001" />
       <inertia
         ixx="0.00017957425901848"
@@ -439,5 +508,5 @@
       rpy="1.5708 0 -3.1416" />
     <parent
-      link="base_link" />
+      link="robot_base" /> <!-- original : base_link -->
     <child
       link="wheel2.2_Link" />
@@ -457,5 +526,5 @@
         rpy="0 0 0" />
       <mass
-        value="0.240893303086836" />
+        value="0.0001" />
       <inertia
         ixx="0.000105035118852508"
@@ -497,5 +566,5 @@
       rpy="1.5708 0 -3.1416" />
     <parent
-      link="base_link" />
+      link="robot_base" /> <!-- original : base_link -->
     <child
       link="wheel2.3_Link" />
@@ -515,5 +584,5 @@
         rpy="0 0 0" />
       <mass
-        value="1.35828296445862" />
+        value="0.0001" />
       <inertia
         ixx="0.00232456013775523"
@@ -555,5 +624,5 @@
       rpy="1.5708 0 -3.1416" />
     <parent
-      link="base_link" />
+      link="robot_base" /> <!-- original : base_link -->
     <child
       link="wheel3_Link" />
@@ -573,5 +642,5 @@
         rpy="0 0 0" />
       <mass
-        value="0.271192811687251" />
+        value="0.0001" />
       <inertia
         ixx="0.000179574259018481"
@@ -613,5 +682,5 @@
       rpy="1.5708 0 -3.1416" />
     <parent
-      link="base_link" />
+      link="robot_base" /> <!-- original : base_link -->
     <child
       link="wheel3.1_Link" />
@@ -631,5 +700,5 @@
         rpy="0 0 0" />
       <mass
-        value="0.27119281168725" />
+        value="0.0001" />
       <inertia
         ixx="0.00017957425901848"
@@ -671,5 +740,5 @@
       rpy="1.5708 0 -3.1416" />
     <parent
-      link="base_link" />
+      link="robot_base" /> <!-- original : base_link -->
     <child
       link="wheel3.2_Link" />
@@ -689,5 +758,5 @@
         rpy="0 0 0" />
       <mass
-        value="0.245836054976119" />
+        value="0.0001" />
       <inertia
         ixx="0.000105264944409738"
@@ -729,5 +798,5 @@
       rpy="1.5708 0 -3.1416" />
     <parent
-      link="base_link" />
+      link="robot_base" /> <!-- original : base_link -->
     <child
       link="wheel3.3_Link" />
@@ -747,5 +816,5 @@
         rpy="0 0 0" />
       <mass
-        value="1.35828296445862" />
+        value="0.0001" />
       <inertia
         ixx="0.00232456564213727"
@@ -787,5 +856,5 @@
       rpy="1.5708 0 -3.1416" />
     <parent
-      link="base_link" />
+      link="robot_base" /> <!-- original : base_link -->
     <child
       link="wheel4_Link" />
@@ -805,5 +874,5 @@
         rpy="0 0 0" />
       <mass
-        value="0.271192811687251" />
+        value="0.0001" />
       <inertia
         ixx="0.000179574259018481"
@@ -845,5 +914,5 @@
       rpy="1.5708 0 -3.1416" />
     <parent
-      link="base_link" />
+      link="robot_base" /> <!-- original : base_link -->
     <child
       link="wheel4.1_Link" />
@@ -863,5 +932,5 @@
         rpy="0 0 0" />
       <mass
-        value="0.27119281168725" />
+        value="0.0001" />
       <inertia
         ixx="0.00017957425901848"
@@ -903,5 +972,5 @@
       rpy="1.5708 0 -3.1416" />
     <parent
-      link="base_link" />
+      link="robot_base" /> <!-- original : base_link -->
     <child
       link="wheel4.2_Link" />
@@ -921,5 +990,5 @@
         rpy="0 0 0" />
       <mass
-        value="0.245836054976119" />
+        value="0.0001" />
       <inertia
         ixx="0.000105264944409738"
@@ -961,5 +1030,5 @@
       rpy="1.5708 0 -3.1416" />
     <parent
-      link="base_link" />
+      link="robot_base" /> <!-- original : base_link -->
     <child
       link="wheel4.3_Link" />
@@ -972,3 +1041,194 @@
       velocity="0" />
   </joint>
+  <!-- add joint frame stand 13 Nov 23-->
+<!--  <joint name="baseto_framestand" type="fixed">
+    <origin rpy="0 0 0" xyz="0.3 0 0"/>
+    <parent link="robot_base"/>
+    <child link="rbot_base2"/>
+  </joint> -->
+<!-- original joint r200 camera to bunker -->
+<!--  <joint name="camera_joint" type="fixed">
+    <origin xyz="0.064 -0.065 0.094" rpy="0 0 0"/>
+    <parent link="robot_base"/> <!-original base link ->
+    <child link="camera_link"/>
+  </joint> -->
+  <link name="camera_link">
+    <visual>
+     <origin xyz="0 0 0" rpy="1.57 0 1.57"/>
+      <geometry>
+       <mesh filename="package://bunker_description/meshes/sensors/r200.dae" />
+      </geometry>
+    </visual>
+    <collision>
+      <origin xyz="0.003 0.065 0.007" rpy="0 0 0"/>
+      <geometry>
+        <box size="0.012 0.132 0.020"/>
+      </geometry>
+    </collision>
+    <!-- This inertial field needs doesn't contain reliable data!! -->
+<!--   <inertial>
+      <mass value="0.564" />
+      <origin xyz="0 0 0" />
+      <inertia ixx="0.003881243" ixy="0.0" ixz="0.0"
+               iyy="0.000498940" iyz="0.0"
+               izz="0.003879257" />
+    </inertial>-->
+  </link>
+  <joint name="camera_rgb_joint" type="fixed">
+    <origin xyz="${r200_cam_rgb_px} ${r200_cam_rgb_py} ${r200_cam_rgb_pz}" rpy="0 0 0"/>
+    <parent link="camera_link"/>
+    <child link="camera_rgb_frame"/>
+  </joint>
+  <link name="camera_rgb_frame"/>
+  <joint name="camera_rgb_optical_joint" type="fixed">
+    <origin xyz="0 0 0" rpy="-1.57 0 -1.57"/>
+    <parent link="camera_rgb_frame"/>
+    <child link="camera_rgb_optical_frame"/>
+  </joint>
+  <link name="camera_rgb_optical_frame"/>
+  <joint name="camera_depth_joint" type="fixed">
+    <origin xyz="${r200_cam_rgb_px} ${r200_cam_rgb_py + r200_cam_depth_offset} ${r200_cam_rgb_pz}" rpy="0 0 0"/>
+    <parent link="camera_link"/>
+    <child link="camera_depth_frame"/>
+  </joint>
+  <link name="camera_depth_frame"/>
+  <joint name="camera_depth_optical_joint" type="fixed">
+    <origin xyz="0 0 0" rpy="-1.57 0 -1.57"/>
+    <parent link="camera_depth_frame"/>
+    <child link="camera_depth_optical_frame"/>
+  </joint>
+  <link name="camera_depth_optical_frame"/>
+  <!-- from waffle models sdf from pkg=turtlebot3_simulation-->
+  <!-- <link name="image">
+    <inertial>
+      <pose>-0.069 0 0.104 0 0 0</pose>
+      <inertia>
+        <ixx>0.001</ixx>
+        <ixy>0.000</ixy>
+        <ixz>0.000</ixz>
+        <iyy>0.001</iyy>
+        <iyz>0.000</iyz>
+        <izz>0.001</izz>
+      </inertia>
+      <mass>0.035</mass>
+    </inertial>
+    <collision name="image_collision">
+      <pose>-0.069 0 0.104 0 0 0</pose>
+      <geometry>
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