Commit message: updated from bunker_sim and world map

File: bunker_explorer_bot/bunker_explorer_description/urdf/bunker_camera_base-footprint_real.xacro (robot description, xacro)
@@ -1307,13 +1307,13 @@
       <!--<robotNamespace>$(arg robot_namespace)</robotNamespace> -->
       <updateRate>40</updateRate>
-      <bodyName>robot_base</bodyName>
-      <frameId>robot_base</frameId>
+      <bodyName>gps_link</bodyName>
+      <frameId>gps_link</frameId>
       <topicName>ublox_gps/fix</topicName> <!-- original navsat/fix-->
       <velocityTopicName>ublox_gps/vel</velocityTopicName> <!-- original navsat/vel-->
-      <referenceLatitude>49.9</referenceLatitude>
-      <referenceLongitude>8.9</referenceLongitude>
+      <referenceLatitude>37.871112</referenceLatitude>
+      <referenceLongitude>127.746019</referenceLongitude>
       <referenceHeading>0</referenceHeading>
       <referenceAltitude>0</referenceAltitude>
-      <drift>0.0001 0.0001 0.0001</drift>
+      <drift>0.001 0.001 0.001</drift>
     </plugin>
   </gazebo>
@@ -1323,6 +1323,6 @@
       <robotNamespace>/</robotNamespace>
       <updateRate>50.0</updateRate>
-      <bodyName>camera_link</bodyName> <!--original base_link-->
-      <!--frameId>imu_link</fameId-->
+      <bodyName>imu_link</bodyName> <!--original base_link-->
+      <frameId>imu_link</fameId>
       <topicName>imu/data</topicName>
       <accelDrift>0.005 0.005 0.005</accelDrift>

File: bunker_explorer_bot/bunker_explorer_description/urdf/bunker_camera_base-footprint_rev0.xacro (robot description, xacro)
@@ -58,10 +58,10 @@
     </visual>
   </link>
-  <joint name="base_to_Servo_B2" type="fixed">
+ <joint name="base_to_Servo_B2" type="fixed">
     <parent link="rbot_base2"/>
     <child link="servo_bottom2"/>
     <origin xyz="0 0 0.14"/>
   </joint>
-  <joint name="servo_bottom_to_up_mount2" type="fixed">
+ <joint name="servo_bottom_to_up_mount2" type="fixed">
     <parent link="servo_bottom2"/>
     <child link="up_mount2"/>
@@ -75,61 +75,62 @@
 <!-- add frame stand joint gps 19Nov23 -->
   <joint name="baseto_framestand_gps" type="fixed">
-    <origin rpy="0 0 0" xyz="-0.25 0 0"/>
-    <parent link="robot_base"/>
-    <child link="rbot_base3"/>
+	<origin rpy="0 0 0" xyz="-0.25 0 0"/>
+	<parent link="robot_base"/>
+	<child link="rbot_base3"/>
   </joint>
   <link name="rbot_base3">
-    <visual>
-      <geometry>
-        <box size="0.045 0.09 0.03"/>
-      </geometry>
-      <origin rpy="0 0 0" xyz="0 0 0"/>
-      <material name="red"/>
-    </visual>
+	<visual>
+  	<geometry>
+    	<box size="0.045 0.09 0.03"/>
+  	</geometry>
+  	<origin rpy="0 0 0" xyz="0 0 0"/>
+  	<material name="red"/>
+	</visual>
   </link>
   <link name="servo_bottom3">
-    <visual>
-      <geometry>
-        <cylinder length="0.25" radius="0.015"/>
-      </geometry>
-      <origin rpy="0 0 0" xyz="0 0 0"/>
-      <material name="green"/>
-    </visual>
+	<visual>
+  	<geometry>
+    	<cylinder length="0.25" radius="0.015"/>
+  	</geometry>
+  	<origin rpy="0 0 0" xyz="0 0 0"/>
+  	<material name="green"/>
+	</visual>
   </link>
   <link name="up_mount3">
-    <visual>
-      <geometry>
-        <box size="0.05 0.148 0.05"/>
-      </geometry>
-      <origin rpy="0 0. 0" xyz="0 0 0"/>
-      <material name="blue"/>
-    </visual>
+	<visual>
+  	<geometry>
+    	<box size="0.05 0.148 0.05"/>
+  	</geometry>
+  	<origin rpy="0 0. 0" xyz="0 0 0"/>
+  	<material name="blue"/>
+	</visual>
   </link>
   <link name="gps_link">
-    <visual>
-      <geometry>
-        <cylinder length="0.065" radius="0.075"/>
-      </geometry>
-      <origin rpy="0 0 0" xyz="0 0 0"/>
-      <material name="green"/>
-    </visual>
-  </link>
-  <joint name="base_to_gps" type="fixed">
-    <parent link="rbot_base3"/>
-    <child link="servo_bottom3"/>
-    <origin xyz="0 0 0.14"/>
-  </joint>
-  <joint name="servo_bottom_to_up_mount3" type="fixed">
-    <parent link="servo_bottom3"/>
-    <child link="up_mount3"/>
-    <origin xyz="0 0 0.15"/>
+	<visual>
+  	<geometry>
+    	<cylinder length="0.065" radius="0.075"/>
+  	</geometry>
+  	<origin rpy="0 0 0" xyz="0 0 0"/>
+  	<material name="green"/>
+	</visual>
+  </link>
+ <joint name="base_to_gps" type="fixed">
+	<parent link="rbot_base3"/>
+	<child link="servo_bottom3"/>
+	<origin xyz="0 0 0.14"/>
+  </joint>
+ <joint name="servo_bottom_to_up_mount3" type="fixed">
+	<parent link="servo_bottom3"/>
+	<child link="up_mount3"/>
+	<origin xyz="0 0 0.15"/>
   </joint>
   <joint name="mount_to_gps" type="fixed">
-    <parent link="up_mount3"/>
-    <child link="gps_link"/> <!-- original: base_link -->
-    <origin rpy="0 0 0" xyz="0.0 0.0 0.0"/>
+	<parent link="up_mount3"/>
+	<child link="gps_link"/> <!-- original: base_link -->
+	<origin rpy="0 0 0" xyz="0.0 0.0 0.0"/>
   </joint>
 <!--  ======= End of editing on 19 Nov 23 ======== -->
-  <link name="robot_base"> <!--original : base_link -->
+  <link
+    name="robot_base"> <!--original : base_link -->
      <inertial>
       <origin
@@ -170,5 +171,6 @@
     </collision>
   </link>
-  <link name="wheel1_Link">
+  <link
+    name="wheel1_Link">
     <inertial>
       <origin
@@ -209,5 +211,6 @@
     </collision>
   </link>
-  <joint name="wheel1_joint"
+  <joint
+    name="wheel1_joint"
     type="revolute">
     <origin
@@ -226,5 +229,6 @@
       velocity="0" />
   </joint>
-  <link name="wheel1.1_Link">
+  <link
+    name="wheel1.1_Link">
     <inertial>
       <origin
@@ -265,5 +269,6 @@
     </collision>
   </link>
-  <joint name="wheel1.1_jont"
+  <joint
+    name="wheel1.1_jont"
     type="revolute">
     <origin
@@ -282,5 +287,6 @@
       velocity="0" />
   </joint>
-  <link name="wheel1.2_Link">
+  <link
+    name="wheel1.2_Link">
     <inertial>
       <origin
@@ -321,5 +327,6 @@
     </collision>
   </link>
-  <joint name="wheel1.2_joint"
+  <joint
+    name="wheel1.2_joint"
     type="revolute">
     <origin
@@ -338,5 +345,6 @@
       velocity="0" />
   </joint>
-  <link name="wheel1.3_Link">
+  <link
+    name="wheel1.3_Link">
     <inertial>
       <origin
@@ -377,5 +385,6 @@
     </collision>
   </link>
-  <joint name="wheel1.3_joint"
+  <joint
+    name="wheel1.3_joint"
     type="revolute">
     <origin
@@ -394,5 +403,6 @@
       velocity="0" />
   </joint>
-  <link name="wheel2_Link">
+  <link
+    name="wheel2_Link">
     <inertial>
       <origin
@@ -433,5 +443,6 @@
     </collision>
   </link>
-  <joint name="wheel2_joint"
+  <joint
+    name="wheel2_joint"
     type="revolute">
     <origin
@@ -450,5 +461,6 @@
       velocity="0" />
   </joint>
-  <link name="wheel2.1_Link">
+  <link
+    name="wheel2.1_Link">
     <inertial>
       <origin
@@ -489,5 +501,6 @@
     </collision>
   </link>
-  <joint name="wheel2.1_joint"
+  <joint
+    name="wheel2.1_joint"
     type="revolute">
     <origin
@@ -506,5 +519,6 @@
       velocity="0" />
   </joint>
-  <link name="wheel2.2_Link">
+  <link
+    name="wheel2.2_Link">
     <inertial>
       <origin
@@ -545,5 +559,6 @@
     </collision>
   </link>
-  <joint name="wheel2.2_joint"
+  <joint
+    name="wheel2.2_joint"
     type="revolute">
     <origin
@@ -562,5 +577,6 @@
       velocity="0" />
   </joint>
-  <link name="wheel2.3_Link">
+  <link
+    name="wheel2.3_Link">
     <inertial>
       <origin
@@ -601,5 +617,6 @@
     </collision>
   </link>
-  <joint name="wheel2.3_joint"
+  <joint
+    name="wheel2.3_joint"
     type="revolute">
     <origin
@@ -618,5 +635,6 @@
       velocity="0" />
   </joint>
-  <link name="wheel3_Link">
+  <link
+    name="wheel3_Link">
     <inertial>
       <origin
@@ -657,5 +675,6 @@
     </collision>
   </link>
-  <joint name="wheel3_joint"
+  <joint
+    name="wheel3_joint"
     type="revolute">
     <origin
@@ -674,5 +693,6 @@
       velocity="0" />
   </joint>
-  <link name="wheel3.1_Link">
+  <link
+    name="wheel3.1_Link">
     <inertial>
       <origin
@@ -713,5 +733,6 @@
     </collision>
   </link>
-  <joint name="wheel3.1_joint"
+  <joint
+    name="wheel3.1_joint"
     type="revolute">
     <origin
@@ -730,5 +751,6 @@
       velocity="0" />
   </joint>
-  <link name="wheel3.2_Link">
+  <link
+    name="wheel3.2_Link">
     <inertial>
       <origin
@@ -787,5 +809,6 @@
       velocity="0" />
   </joint>
-  <link name="wheel3.3_Link">
+  <link
+    name="wheel3.3_Link">
     <inertial>
       <origin
@@ -826,5 +849,6 @@
     </collision>
   </link>
-  <joint name="wheel3.3_joint"
+  <joint
+    name="wheel3.3_joint"
     type="revolute">
     <origin
@@ -843,5 +867,6 @@
       velocity="0" />
   </joint>
-  <link name="wheel4_Link">
+  <link
+    name="wheel4_Link">
     <inertial>
       <origin
@@ -882,5 +907,6 @@
     </collision>
   </link>
-  <joint name="wheel4_joint"
+  <joint
+    name="wheel4_joint"
     type="revolute">
     <origin
@@ -899,5 +925,6 @@
       velocity="0" />
   </joint>
-  <link name="wheel4.1_Link">
+  <link
+    name="wheel4.1_Link">
     <inertial>
       <origin
@@ -938,5 +965,6 @@
     </collision>
   </link>
-  <joint name="wheel4.1_joint"
+  <joint
+    name="wheel4.1_joint"
     type="revolute">
     <origin
@@ -955,5 +983,6 @@
       velocity="0" />
   </joint>
-  <link name="wheel4.2_Link">
+  <link
+    name="wheel4.2_Link">
     <inertial>
       <origin
@@ -994,5 +1023,6 @@
     </collision>
   </link>
-  <joint name="wheel4.2_joint"
+  <joint
+    name="wheel4.2_joint"
     type="revolute">
     <origin
@@ -1011,5 +1041,6 @@
       velocity="0" />
   </joint>
-  <link name="wheel4.3_Link">
+  <link
+    name="wheel4.3_Link">
     <inertial>
       <origin
@@ -1050,5 +1081,6 @@
     </collision>
   </link>
-  <joint name="wheel4.3_joint"
+  <joint
+    name="wheel4.3_joint"
     type="revolute">
     <origin
@@ -1166,32 +1198,4 @@
     </sensor>
   </link> -->
- <!-- ====== add imu link on 19 nov23 ====== -->
-  <link name="imu_link">
-    <visual>
-      <geometry>
-        <box size="0.05 0.02 0.02"/>
-      </geometry>
-      <material name="red"/>
-    </visual>
-  </link>
-  <joint name="imu_joint" type="fixed">
-    <origin rpy="0 0 0" xyz="-0.025 -0.015 0.005"/>
-    <parent link="camera_link"/>
-    <child link="imu_link"/>
-  </joint>
- <!-- ====== add imu link2 on 19 nov23 ====== -->
-  <link name="imu_link2">
-    <visual>
-      <geometry>
-        <box size="0.05 0.026 0.005"/>
-      </geometry>
-      <material name="red"/>
-    </visual>
-  </link>
-  <joint name="imu_joint2" type="fixed">
-	  <origin rpy="0 0 0" xyz="0.0 0.0 0.001"/>
-	  <parent link="robot_base"/>
-	  <child link="imu_link2"/>
-  </joint>
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
File: bunker_explorer_bot/bunker_explorer_description/urdf/bunker_camera_base-footprint_sim.xacro (robot description, xacro)
@@ -130,5 +130,5 @@
     <origin rpy="0 0 0" xyz="0.0 0.0 0.0"/>
   </joint>
-<!--  ======= End of editing on 19 Nov 23 ======== -->
+<!--  ======= End of gps urdf editing on 19 Nov 23 ======== -->
   <link name="robot_base"> <!--original : base_link -->
      <inertial>
@@ -1081,5 +1081,5 @@
   <link name="camera_link">
     <visual>
-     <origin xyz="0 0 0" rpy="1.57 0 1.57"/>
+       <origin xyz="0 0 0" rpy="1.57 0 1.57"/>
       <geometry>
        <mesh filename="package://bunker_description/meshes/sensors/r200.dae" />
@@ -1194,4 +1194,5 @@
 	  <child link="imu_link2"/>
   </joint>
+ <!-- ====== end of editing imu link 1 and 2 on 19 nov23 ====== -->
   <!-- /////////////////////////////////   gazebo color   ////////////////////////////////////// -->
  <gazebo reference="robot_base"> <!--base_link-->
@@ -1291,6 +1292,6 @@
       <robotNamespace>/</robotNamespace>
       <updateRate>50.0</updateRate>
-      <bodyName>camera_link</bodyName> <!--original base_link-->
-      <!--frameId>imu_link</fameId-->
+      <bodyName>imu_link</bodyName> <!--original base_link-->
+      <frameId>imu_link</frameId>
       <topicName>imu/data</topicName>
       <accelDrift>0.005 0.005 0.005</accelDrift>

File: bunker_explorer_bot/bunker_explorer_description/urdf/bunker_camera_base-footprint_sim_rev0.xacro (robot description, xacro)
@@ -4,8 +4,4 @@
      For more information, please see http://wiki.ros.org/sw_urdf_exporter -->
 <robot  name="bunker_realsense_description" xmlns:xacro="http://www.ros.org/wiki/xacro">
-  <xacro:property name="r200_cam_rgb_px" value="0.005"/>
-  <xacro:property name="r200_cam_rgb_py" value="0.018"/>
-  <xacro:property name="r200_cam_rgb_pz" value="0.013"/>
-  <xacro:property name="r200_cam_depth_offset" value="0.01"/>
   <xacro:arg name="camera_visual" default="false"/>
   <link name="base_footprint"/>
@@ -63,5 +59,5 @@
     <origin xyz="0 0 0.14"/>
   </joint>
-  <joint name="servo_bottom_to_up_mount2" type="fixed">
+ <joint name="servo_bottom_to_up_mount2" type="fixed">
     <parent link="servo_bottom2"/>
     <child link="up_mount2"/>
@@ -70,6 +66,6 @@
   <joint name="mount_to_camera2" type="fixed">
     <parent link="up_mount2"/>
-    <child link="camera_link"/> <!-- original: base_link -->
-    <origin rpy="0 0 0" xyz="0.03 -0.065 0.00"/>
+    <child link="base_link"/> <!-- original: base_link -->
+    <origin rpy="0 0 0" xyz="0.03 -0.0 0.00"/>
   </joint>
 <!-- add frame stand joint gps 19Nov23 -->
@@ -80,38 +76,38 @@
   </joint>
   <link name="rbot_base3">
-    <visual>
-      <geometry>
-        <box size="0.045 0.09 0.03"/>
-      </geometry>
-      <origin rpy="0 0 0" xyz="0 0 0"/>
-      <material name="red"/>
-    </visual>
+	<visual>
+  	<geometry>
+    	<box size="0.045 0.09 0.03"/>
+  	</geometry>
+  	<origin rpy="0 0 0" xyz="0 0 0"/>
+  	<material name="red"/>
+	</visual>
   </link>
   <link name="servo_bottom3">
-    <visual>
-      <geometry>
-        <cylinder length="0.25" radius="0.015"/>
-      </geometry>
-      <origin rpy="0 0 0" xyz="0 0 0"/>
-      <material name="green"/>
-    </visual>
+	<visual>
+  	<geometry>
+    	<cylinder length="0.25" radius="0.015"/>
+  	</geometry>
+  	<origin rpy="0 0 0" xyz="0 0 0"/>
+  	<material name="green"/>
+	</visual>
   </link>
   <link name="up_mount3">
-    <visual>
-      <geometry>
-        <box size="0.05 0.148 0.05"/>
-      </geometry>
-      <origin rpy="0 0. 0" xyz="0 0 0"/>
-      <material name="blue"/>
-    </visual>
+	<visual>
+  	<geometry>
+    	<box size="0.05 0.148 0.05"/>
+  	</geometry>
+  	<origin rpy="0 0. 0" xyz="0 0 0"/>
+  	<material name="blue"/>
+	</visual>
   </link>
   <link name="gps_link">
-    <visual>
-      <geometry>
-        <cylinder length="0.065" radius="0.075"/>
-      </geometry>
-      <origin rpy="0 0 0" xyz="0 0 0"/>
-      <material name="green"/>
-    </visual>
+	<visual>
+  	<geometry>
+    	<cylinder length="0.065" radius="0.075"/>
+  	</geometry>
+  	<origin rpy="0 0 0" xyz="0 0 0"/>
+  	<material name="green"/>
+	</visual>
   </link>
   <joint name="base_to_gps" type="fixed">
@@ -130,6 +126,7 @@
     <origin rpy="0 0 0" xyz="0.0 0.0 0.0"/>
   </joint>
-<!--  ======= End of editing on 19 Nov 23 ======== -->
-  <link name="robot_base"> <!--original : base_link -->
+<!--  ======= End of gps urdf editing on 19 Nov 23 ======== -->
+  <link
+    name="robot_base"> <!--original : base_link -->
      <inertial>
       <origin
@@ -170,5 +167,6 @@
     </collision>
   </link>
-  <link name="wheel1_Link">
+  <link
+    name="wheel1_Link">
     <inertial>
       <origin
@@ -209,5 +207,6 @@
     </collision>
   </link>
-  <joint name="wheel1_joint"
+  <joint
+    name="wheel1_joint"
     type="revolute">
     <origin
@@ -226,5 +225,6 @@
       velocity="0" />
   </joint>
-  <link name="wheel1.1_Link">
+  <link
+    name="wheel1.1_Link">
     <inertial>
       <origin
@@ -265,5 +265,6 @@
     </collision>
   </link>
-  <joint name="wheel1.1_jont"
+  <joint
+    name="wheel1.1_jont"
     type="revolute">
     <origin
@@ -282,5 +283,6 @@
       velocity="0" />
   </joint>
-  <link name="wheel1.2_Link">
+  <link
+    name="wheel1.2_Link">
     <inertial>
       <origin
@@ -321,5 +323,6 @@
     </collision>
   </link>
-  <joint name="wheel1.2_joint"
+  <joint
+    name="wheel1.2_joint"
     type="revolute">
     <origin
@@ -338,5 +341,6 @@
       velocity="0" />
   </joint>
-  <link name="wheel1.3_Link">
+  <link
+    name="wheel1.3_Link">
     <inertial>
       <origin
@@ -377,5 +381,6 @@
     </collision>
   </link>
-  <joint name="wheel1.3_joint"
+  <joint
+    name="wheel1.3_joint"
     type="revolute">
     <origin
@@ -394,5 +399,6 @@
       velocity="0" />
   </joint>
-  <link name="wheel2_Link">
+  <link
+    name="wheel2_Link">
     <inertial>
       <origin
@@ -433,5 +439,6 @@
     </collision>
   </link>
-  <joint name="wheel2_joint"
+  <joint
+    name="wheel2_joint"
     type="revolute">
     <origin
@@ -450,5 +457,6 @@
       velocity="0" />
   </joint>
-  <link name="wheel2.1_Link">
+  <link
+    name="wheel2.1_Link">
     <inertial>
       <origin
@@ -489,5 +497,6 @@
     </collision>
   </link>
-  <joint name="wheel2.1_joint"
+  <joint
+    name="wheel2.1_joint"
     type="revolute">
     <origin
@@ -506,5 +515,6 @@
       velocity="0" />
   </joint>
-  <link name="wheel2.2_Link">
+  <link
+    name="wheel2.2_Link">
     <inertial>
       <origin
@@ -545,5 +555,6 @@
     </collision>
   </link>
-  <joint name="wheel2.2_joint"
+  <joint
+    name="wheel2.2_joint"
     type="revolute">
     <origin
@@ -562,5 +573,6 @@
       velocity="0" />
   </joint>
-  <link name="wheel2.3_Link">
+  <link
+    name="wheel2.3_Link">
     <inertial>
       <origin
@@ -601,5 +613,6 @@
     </collision>
   </link>
-  <joint name="wheel2.3_joint"
+  <joint
+    name="wheel2.3_joint"
     type="revolute">
     <origin
@@ -618,5 +631,6 @@
       velocity="0" />
   </joint>
-  <link name="wheel3_Link">
+  <link
+    name="wheel3_Link">
     <inertial>
       <origin
@@ -657,5 +671,6 @@
     </collision>
   </link>
-  <joint name="wheel3_joint"
+  <joint
+    name="wheel3_joint"
     type="revolute">
     <origin
@@ -674,5 +689,6 @@
       velocity="0" />
   </joint>
-  <link name="wheel3.1_Link">
+  <link
+    name="wheel3.1_Link">
     <inertial>
       <origin
@@ -713,5 +729,6 @@
     </collision>
   </link>
-  <joint name="wheel3.1_joint"
+  <joint
+    name="wheel3.1_joint"
     type="revolute">
     <origin
@@ -730,5 +747,6 @@
       velocity="0" />
   </joint>
-  <link name="wheel3.2_Link">
+  <link
+    name="wheel3.2_Link">
     <inertial>
       <origin
@@ -787,5 +805,6 @@
       velocity="0" />
   </joint>
-  <link name="wheel3.3_Link">
+  <link
+    name="wheel3.3_Link">
     <inertial>
       <origin
@@ -826,5 +845,6 @@
     </collision>
   </link>
-  <joint name="wheel3.3_joint"
+  <joint
+    name="wheel3.3_joint"
     type="revolute">
     <origin
@@ -843,5 +863,6 @@
       velocity="0" />
   </joint>
-  <link name="wheel4_Link">
+  <link
+    name="wheel4_Link">
     <inertial>
       <origin
@@ -882,5 +903,6 @@
     </collision>
   </link>
-  <joint name="wheel4_joint"
+  <joint
+    name="wheel4_joint"
     type="revolute">
     <origin
@@ -899,5 +921,6 @@
       velocity="0" />
   </joint>
-  <link name="wheel4.1_Link">
+  <link
+    name="wheel4.1_Link">
     <inertial>
       <origin
@@ -938,5 +961,6 @@
     </collision>
   </link>
-  <joint name="wheel4.1_joint"
+  <joint
+    name="wheel4.1_joint"
     type="revolute">
     <origin
@@ -955,5 +979,6 @@
       velocity="0" />
   </joint>
-  <link name="wheel4.2_Link">
+  <link
+    name="wheel4.2_Link">
     <inertial>
       <origin
@@ -994,5 +1019,6 @@
     </collision>
   </link>
-  <joint name="wheel4.2_joint"
+  <joint
+    name="wheel4.2_joint"
     type="revolute">
     <origin
@@ -1011,5 +1037,6 @@
       velocity="0" />
   </joint>
-  <link name="wheel4.3_Link">
+  <link
+    name="wheel4.3_Link">
     <inertial>
       <origin
@@ -1050,5 +1077,6 @@
     </collision>
   </link>
-  <joint name="wheel4.3_joint"
+  <joint
+    name="wheel4.3_joint"
     type="revolute">
     <origin
@@ -1067,52 +1095,48 @@
       velocity="0" />
   </joint>
-  <!-- add joint frame stand 13 Nov 23-->
-<!--  <joint name="baseto_framestand" type="fixed">
-    <origin rpy="0 0 0" xyz="0.3 0 0"/>
-    <parent link="robot_base"/>
-    <child link="rbot_base2"/>
-  </joint> -->
-<!-- original joint r200 camera to bunker -->
-<!--  <joint name="camera_joint" type="fixed">
-    <origin xyz="0.064 -0.065 0.094" rpy="0 0 0"/>
-    <parent link="robot_base"/> <!-original base link ->
+<!-- =======add realsense d435i real camera plugin edited on 19nov23 ========= -->
+  <material name="aluminum">
+	  <color rgba="0.5 0.5 0.5 1"/>
+  </material>
+  <material name="plastic">
+	  <color rgba="0.1 0.1 0.1 1"/>
+  </material>
+  <link name="base_link"/>
+  <!-- camera body, with origin at bottom screw mount -->
+  <joint name="camera_joint" type="fixed">
+    <origin rpy="0 0 0" xyz="0 0 0"/>
+    <parent link="base_link"/>
+    <child link="camera_bottom_screw_frame"/>
+  </joint>
+  <link name="camera_bottom_screw_frame"/>
+  <joint name="camera_link_joint" type="fixed">
+    <origin rpy="0 0 0" xyz="0.0106 0.0175 0.0125"/>
+    <parent link="camera_bottom_screw_frame"/>
     <child link="camera_link"/>
-  </joint> -->
+  </joint>
   <link name="camera_link">
     <visual>
-     <origin xyz="0 0 0" rpy="1.57 0 1.57"/>
-      <geometry>
-       <mesh filename="package://bunker_description/meshes/sensors/r200.dae" />
-      </geometry>
-    </visual>
-    <collision>
-      <origin xyz="0.003 0.065 0.007" rpy="0 0 0"/>
-      <geometry>
-        <box size="0.012 0.132 0.020"/>
-      </geometry>
-    </collision>
-    <!-- This inertial field needs doesn't contain reliable data!! -->
-<!--   <inertial>
-      <mass value="0.564" />
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