Commit message: updated bunker_explorer_ws

File: bunker_explorer_bot/bunker_explorer_description/urdf/bunker_realsense.urdf.xacro (robot description, xacro)
@@ -182,5 +182,5 @@
       <material name="blue"/>
     </visual>
-  </link> -->
+  </link> <!-- -->
     <!-- added new joint-->
  <!--<joint name="base_to_Servo_B2" type="fixed">
